File: main.brd (EAGLE design)
At the start: 160 x 100 mm, 0 parts

Commit message: Add files via upload
Parts:
- added U1: ATMEGA328P-AU, Downloads:QFP80P900X900X120-32N
- added U2: DRV8833PWPR, Downloads:PWP16_2P31X2P46
Connections:
- new net AVCC: U1.18
- new net GND: U1.21, U1.3, U1.5, U2.13
- new net VCC: U1.4, U1.6
- new net VINT: U2.14
- new net VM: U2.12
Changed lines of the file:
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@@
 <layer number="48" name="Document" color="7" fill="1" visible="yes" active="yes"/>
 <layer number="49" name="Reference" color="7" fill="1" visible="yes" active="yes"/>
+<layer number="50" name="dxf" color="12" fill="1" visible="no" active="no"/>
 <layer number="51" name="tDocu" color="7" fill="1" visible="yes" active="yes"/>
 <layer number="52" name="bDocu" color="7" fill="1" visible="yes" active="yes"/>
+<layer number="53" name="tGND_GNDA" color="7" fill="1" visible="no" active="no"/>
+<layer number="54" name="bGND_GNDA" color="7" fill="1" visible="no" active="no"/>
+<layer number="56" name="wert" color="7" fill="1" visible="no" active="no"/>
+<layer number="57" name="tCAD" color="7" fill="1" visible="no" active="no"/>
 <layer number="88" name="SimResults" color="9" fill="1" visible="no" active="no"/>
 <layer number="89" name="SimProbes" color="9" fill="1" visible="no" active="no"/>
@@
 <layer number="97" name="Info" color="7" fill="1" visible="no" active="no"/>
 <layer number="98" name="Guide" color="6" fill="1" visible="no" active="no"/>
+<layer number="99" name="SpiceOrder" color="7" fill="1" visible="no" active="no"/>
+<layer number="100" name="Muster" color="7" fill="1" visible="yes" active="yes"/>
+<layer number="101" name="Patch_Top" color="7" fill="1" visible="yes" active="yes"/>
+<layer number="102" name="Vscore" color="7" fill="1" visible="yes" active="yes"/>
+<layer number="103" name="tMap" color="7" fill="1" visible="yes" active="yes"/>
+<layer number="104" name="Name" color="7" fill="1" visible="yes" active="yes"/>
+<layer number="105" name="tPlate" color="7" fill="1" visible="yes" active="yes"/>
+<layer number="106" name="bPlate" color="7" fill="1" visible="yes" active="yes"/>
+<layer number="107" name="Crop" color="7" fill="1" visible="yes" active="yes"/>
+<layer number="108" name="fp8" color="7" fill="1" visible="yes" active="yes"/>
+<layer number="109" name="fp9" color="7" fill="1" visible="yes" active="yes"/>
+<layer number="110" name="fp0" color="7" fill="1" visible="yes" active="yes"/>
+<layer number="111" name="LPC17xx" color="7" fill="1" visible="yes" active="yes"/>
+<layer number="112" name="tSilk" color="7" fill="1" visible="yes" active="yes"/>
+<layer number="113" name="IDFDebug" color="4" fill="1" visible="yes" active="yes"/>
+<layer number="116" name="Patch_BOT" color="7" fill="1" visible="yes" active="yes"/>
+<layer number="121" name="_tsilk" color="7" fill="1" visible="yes" active="yes"/>
+<layer number="122" name="_bsilk" color="7" fill="1" visible="yes" active="yes"/>
+<layer number="123" name="tTestmark" color="7" fill="1" visible="yes" active="yes"/>
+<layer number="124" name="bTestmark" color="7" fill="1" visible="yes" active="yes"/>
+<layer number="125" name="_tNames" color="7" fill="1" visible="yes" active="yes"/>
+<layer number="126" name="_bNames" color="7" fill="1" visible="yes" active="yes"/>
+<layer number="127" name="_tValues" color="7" fill="1" visible="yes" active="yes"/>
+<layer number="128" name="_bValues" color="7" fill="1" visible="yes" active="yes"/>
+<layer number="131" name="tAdjust" color="7" fill="1" visible="yes" active="yes"/>
+<layer number="132" name="bAdjust" color="7" fill="1" visible="yes" active="yes"/>
+<layer number="144" name="Drill_legend" color="7" fill="1" visible="yes" active="yes"/>
+<layer number="150" name="Notes" color="7" fill="1" visible="yes" active="yes"/>
+<layer number="151" name="HeatSink" color="7" fill="1" visible="yes" active="yes"/>
+<layer number="152" name="_bDocu" color="7" fill="1" visible="yes" active="yes"/>
+<layer number="153" name="FabDoc1" color="7" fill="1" visible="yes" active="yes"/>
+<layer number="154" name="FabDoc2" color="7" fill="1" visible="yes" active="yes"/>
+<layer number="155" name="FabDoc3" color="7" fill="1" visible="yes" active="yes"/>
+<layer number="199" name="Contour" color="7" fill="1" visible="yes" active="yes"/>
+<layer number="200" name="200bmp" color="1" fill="10" visible="no" active="no"/>
+<layer number="201" name="201bmp" color="7" fill="1" visible="yes" active="yes"/>
+<layer number="202" name="202bmp" color="7" fill="1" visible="yes" active="yes"/>
+<layer number="203" name="203bmp" color="7" fill="1" visible="yes" active="yes"/>
+<layer number="204" name="204bmp" color="7" fill="1" visible="yes" active="yes"/>
+<layer number="205" name="205bmp" color="7" fill="1" visible="yes" active="yes"/>
+<layer number="206" name="206bmp" color="7" fill="1" visible="yes" active="yes"/>
+<layer number="207" name="207bmp" color="7" fill="1" visible="yes" active="yes"/>
+<layer number="208" name="208bmp" color="7" fill="1" visible="yes" active="yes"/>
+<layer number="209" name="209bmp" color="7" fill="1" visible="yes" active="yes"/>
+<layer number="210" name="210bmp" color="7" fill="1" visible="yes" active="yes"/>
+<layer number="211" name="211bmp" color="7" fill="1" visible="yes" active="yes"/>
+<layer number="212" name="212bmp" color="7" fill="1" visible="yes" active="yes"/>
+<layer number="213" name="213bmp" color="7" fill="1" visible="yes" active="yes"/>
+<layer number="214" name="214bmp" color="7" fill="1" visible="yes" active="yes"/>
+<layer number="215" name="215bmp" color="16" fill="1" visible="yes" active="yes"/>
+<layer number="216" name="216bmp" color="17" fill="1" visible="yes" active="yes"/>
+<layer number="217" name="217bmp" color="18" fill="1" visible="yes" active="yes"/>
+<layer number="218" name="218bmp" color="19" fill="1" visible="yes" active="yes"/>
+<layer number="219" name="219bmp" color="20" fill="1" visible="yes" active="yes"/>
+<layer number="220" name="220bmp" color="21" fill="1" visible="yes" active="yes"/>
+<layer number="221" name="221bmp" color="22" fill="1" visible="yes" active="yes"/>
+<layer number="222" name="222bmp" color="23" fill="1" visible="yes" active="yes"/>
+<layer number="223" name="223bmp" color="24" fill="1" visible="yes" active="yes"/>
+<layer number="224" name="224bmp" color="25" fill="1" visible="yes" active="yes"/>
+<layer number="248" name="Housing" color="7" fill="1" visible="yes" active="yes"/>
+<layer number="249" name="Edge" color="7" fill="1" visible="yes" active="yes"/>
+<layer number="250" name="Descript" color="3" fill="1" visible="no" active="no"/>
+<layer number="251" name="SMDround" color="12" fill="11" visible="no" active="no"/>
+<layer number="254" name="cooling" color="7" fill="1" visible="yes" active="yes"/>
 </layers>
 <board>
@@
 </autorouter>
 <elements>
+<element name="U1" library="Downloads" package="QFP80P900X900X120-32N" value="ATMEGA328P-AU" x="-6.35" y="7.62" smashed="yes">
+<attribute name="DESCRIPTION" value=" Microcontroller Mcu, 8 Bit, Atmega, 20mhz, Tqfp-32 " x="-6.35" y="7.62" size="1.778" layer="27" display="off"/>
+<attribute name="DIGI-KEY_PART_NUMBER" value="ATMEGA328P-AU-ND" x="-6.35" y="7.62" size="1.778" layer="27" display="off"/>
+<attribute name="DIGI-KEY_PURCHASE_URL" value="https://www.digikey.com/product-detail/en/microchip-technology/ATMEGA328P-AU/ATMEGA328P-AU-ND/1832260?utm_source=snapeda&amp;utm_medium=aggregator&amp;utm_campaign=symbol" x="-6.35" y="7.62" size="1.778" layer="27" display="off"/>
+<attribute name="MF" value="Microchip" x="-6.35" y="7.62" size="1.778" layer="27" display="off"/>
+<attribute name="MP" value="ATMEGA328P-AU" x="-6.35" y="7.62" size="1.778" layer="27" display="off"/>
+<attribute name="NAME" x="-11.92938125" y="13.25088125" size="0.814375" layer="25"/>
+<attribute name="PACKAGE" value="TQFP-32 Microchip" x="-6.35" y="7.62" size="1.778" layer="27" display="off"/>
+<attribute name="VALUE" x="-11.87646875" y="1.105440625" size="0.81336875" layer="27"/>
+</element>
+<element name="U2" library="Downloads" package="PWP16_2P31X2P46" value="DRV8833PWPR" x="-7.62" y="-5.08" smashed="yes">
+<attribute name="MANUFACTURER_PART_NUMBER" value="DRV8833PWPR" x="-7.62" y="-5.08" size="1.778" layer="27" display="off"/>
+<attribute name="NAME" x="-10.8966" y="-5.715" size="1.27" layer="25" ratio="6" rot="SR0"/>
+<attribute name="VENDOR" value="Texas Instruments" x="-7.62" y="-5.08" size="1.778" layer="27" display="off"/>
+</element>
 </elements>
 <signals>
+<signal name="VCC">
+<contactref element="U1" pad="4"/>
+<contactref element="U1" pad="6"/>
+<wire x1="-10.65" y1="8.02" x2="-10.65" y2="6.42" width="0" layer="19" extent="1-1"/>
+</signal>
+<signal name="GND">
+<contactref element="U1" pad="3"/>
+<contactref element="U1" pad="21"/>
+<contactref element="U1" pad="5"/>
+<contactref element="U2" pad="13"/>
+<wire x1="-10.65" y1="7.22" x2="-2.05" y2="8.02" width="0" layer="19" extent="1-1"/>
+<wire x1="-10.65" y1="8.82" x2="-10.65" y2="7.22" width="0" layer="19" extent="1-1"/>
+<wire x1="-4.8006" y1="-4.755003125" x2="-2.05" y2="8.02" width="0" layer="19" extent="1-1"/>
+</signal>
+<signal name="AVCC">
+<contactref element="U1" pad="18"/>
+</signal>
+<signal name="VM">
+<contactref element="U2" pad="12"/>
+</signal>
+<signal name="VINT">
+<contactref element="U2" pad="14"/>
+</signal>
 </signals>
 <mfgpreviewcolors>

Commit message: Add files via upload
Parts:
- added C1, C2: (no value), rcl:C0805
- added C3: (no value), rcl:153CLV-0605
- added R1: 0.2, rcl:R0805
- moved U2 59.9 mm to (48.3, 16.5)
- moved U1 52.3 mm to (39.4, 33.0)
Connections:
- removed net VINT: U2.14
- removed net VM: U2.12
- new net N$1: C1.1, U2.14
- new net N$10: U2.8
- new net N$11: U2.2
- new net N$12: U2.4
- new net N$13: U2.5
- new net N$14: U2.7
- new net N$2: C2.2, U2.11
- new net N$3: R1.1, U2.3, U2.6
- new net N$4: C2.1, C3.+, U2.12
- new net N$5: U2.9
- new net N$6: U2.10
- new net N$7: U2.15
- new net N$8: U2.16
- new net N$9: U2.1
- net GND: now also C1.2, C3.-, R1.2, U2.EPAD
Routing:
- added copper zone on layer 1, net GND
- added copper zone on layer 16, net GND
Other:
- board size 160 x 100 mm -> 76.2 x 63.5 mm

Commit message: Add files via upload
Parts:
- added U3: LP2985IM5-5.0, LP2985IM5-5.0:SOT95P284X119-5N
Connections:
- new net VIN: U3.1
Changed lines of the file:
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@@
 <drawing>
 <settings>
-<setting alwaysvectorfont="no"/>
+<setting alwaysvectorfont="yes"/>
 <setting verticaltext="up"/>
 </settings>
@@
 <attribute name="VENDOR" value="Texas Instruments" x="48.26" y="16.51" size="1.778" layer="27" display="off"/>
 </element>
+<element name="U3" library="LP2985IM5-5.0" package="SOT95P284X119-5N" value="LP2985IM5-5.0" x="3.81" y="-7.62" smashed="yes">
+<attribute name="DESCRIPTION" value=" Micropower 150-mA Low-Noise Ultra-Low-Dropout Regulator in SOT-23 and DSBGA Packages 5-SOT-23 -40 to 125 " x="3.81" y="-7.62" size="1.778" layer="27" display="off"/>
+<attribute name="DIGI-KEY_PART_NUMBER" value="LP2985IM5-5.0/NOPBCT-ND" x="3.81" y="-7.62" size="1.778" layer="27" display="off"/>
+<attribute name="DIGI-KEY_PURCHASE_URL" value="https://www.digikey.com/product-detail/en/texas-instruments/LP2985IM5-5.0-NOPB/LP2985IM5-5.0-NOPBCT-ND/334983?utm_source=snapeda&amp;utm_medium=aggregator&amp;utm_campaign=symbol" x="3.81" y="-7.62" size="1.778" layer="27" display="off"/>
+<attribute name="MF" value="Texas Instruments" x="3.81" y="-7.62" size="1.778" layer="27" display="off"/>
+<attribute name="MP" value="LP2985IM5-5.0/NOPB" x="3.81" y="-7.62" size="1.778" layer="27" display="off"/>
+<attribute name="NAME" x="-0.74226875" y="-5.661759375" size="2.0854" layer="25" ratio="10" rot="SR0"/>
+<attribute name="PACKAGE" value="SOT-23 Texas Instruments" x="3.81" y="-7.62" size="1.778" layer="27" display="off"/>
+<attribute name="VALUE" x="-1.862109375" y="-11.68966875" size="2.085709375" layer="27" ratio="10" rot="SR0"/>
+</element>
 </elements>
 <signals>
@@
 <contactref element="U2" pad="7"/>
 </signal>
+<signal name="VIN">
+<contactref element="U3" pad="1"/>
+</signal>
 </signals>

Commit message: Add files via upload
Parts:
- added C10, C11, C8, C9: 100nF, rcl:C0805
- added C4, C5: 1uF, rcl:C0805
- added C6, C7: 20pF, rcl:C0805
- added J1: PJ-015AH-SMT-TR, Downloads:CUI_PJ-015AH-SMT-TR
- added JP1: (no value), pinhead:2X03
- added U4: LP38691DTX-5.0/NOPB, Downloads:TD03B
- added Y1: 16MHz, Downloads:XTAL_ECS-160-20-3X-TR
- C1: value (none) -> 2.2uF
- C2: value (none) -> 10nF
- C3: value (none) -> 10uF
- R1: value 0.2 -> 200m
- U3: value LP2985IM5-5.0 -> LS7366R-TS; device LP2985IM5-5.0:SOT95P284X119-5N -> Downloads:SOP65P640X110-14N
- moved U3 61.4 mm to (57.1, 22.9)
- moved R1 36.9 mm to (40.6, 50.8)
- moved C3 36.9 mm to (68.6, 45.7)
- moved U2 35.7 mm to (50.8, 52.1)
- moved C1 33.0 mm to (61.0, 54.6)
- moved C2 33.0 mm to (61.0, 48.3)
- moved U1 1.27 mm to (38.1, 33.0), turned to 45 degrees
Connections:
- net N$10 renamed !FAULT!
- net N$11 renamed AOUT1
- net N$12 renamed AOUT2
- net N$13 renamed BOUT2
- net N$14 renamed BOUT1
- net N$5 renamed BIN1
- net N$6 renamed BIN2
- net N$7 renamed AIN2
- net N$8 renamed AIN1
- net N$9 renamed !SLEEP!
- removed net AVCC: U1.18
- removed net VCC: U1.4, U1.6
- new net !SS!: JP1.5, U1.17, U3.4
- new net +5V: C10.1, C11.1, C4.1, C8.1, C9.1, JP1.2, U1.18, U1.20, U1.4, U1.6, U3.14, U4.1
- new net ADC: U1.26
- new net MISO: JP1.1, U1.15, U3.6
- new net MOSI: JP1.4, U1.16, U3.7
- new net N$16: C7.1, U1.7, Y1.2
- new net N$18: C6.1, U1.8, Y1.1
- new net RXD: U1.30
- new net SCL: U1.28
- new net SCLK: JP1.3, U1.14, U3.5
- new net SDA: U1.27
- new net TXD: U1.31
- new net VSS: U3.3
- net GND: now also C10.2, C11.2, C4.2, C5.2, C6.2, C7.2, C8.2, C9.2, J1.2, J1.3, JP1.6, U4.4
- net VIN: now also C5.1, J1.1, U4.3; no longer U3.1

Commit message: Add files via upload
Parts:
- removed C11: 100nF, rcl:C0805
- added C12: 100nF, rcl:C0805
- added JP2: (no value), pinhead:2X04
- added JP3, JP4: (no value), pinhead:1X04
- C6, C7: value 20pF -> 22pF
- moved J1 57.2 mm to (66.0, 47.0)
- moved R1 46.9 mm to (66.0, 11.4)
- moved U2 35.2 mm to (66.0, 20.3), turned to 90 degrees
- moved C1 25.7 mm to (64.8, 29.2), turned to 90 degrees
- moved C5 24.2 mm to (49.5, 41.9)
- moved U4 24.1 mm to (47.0, 55.9)
- moved C9 23.3 mm to (31.8, 21.6), turned to 270 degrees
- moved C4 22.9 mm to (43.2, 41.9)
- moved C2 21.6 mm to (71.1, 29.2)
- moved C3 18.1 mm to (57.1, 31.8), turned to 0 degrees
- moved C10 17.3 mm to (31.8, 41.9), turned to 90 degrees
- moved U3 15.3 mm to (45.7, 33.0)
- moved JP1 15.3 mm to (48.3, 6.35), turned to 180 degrees
- moved U1 10.2 mm to (27.9, 31.8), turned to 90 degrees
- moved C6 8.52 mm to (39.4, 11.4)
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Connections:
- new net ENCA: JP4.4, U3.12
- new net ENCB: JP4.3, U3.11
- new net FLOW: JP2.7
- new net RESET: JP1.5, U1.29
- net !SS!: no longer JP1.5
- net +5V: now also JP2.2, JP2.4, JP2.6; no longer C11.1, U1.20
- net ADC: now also JP2.5
- net AIN1: now also U1.1
- net AIN2: now also U1.9
- net AOUT1: now also JP3.4
- net AOUT2: now also JP3.3
- net BIN1: now also U1.10
- net BIN2: now also U1.13
- net BOUT1: now also JP3.1
- net BOUT2: now also JP3.2
- net GND: now also C12.2, JP2.8; no longer C11.2
- net N$4: now also C12.1, U1.20; no longer C2.1, C3.+, U2.12
- net SCL: now also JP2.1
- net SDA: now also JP2.3
- net VIN: now also C2.1, C3.+, U2.12

Commit message: Add files via upload
Parts:
- added B1: (no value), ME507:0805
- added C11: 100nF, rcl:C0805
- added C13: 10nF, rcl:A/3216-18W
- added J3: 1734510-1, Downloads:TE_1734510-1
- added U5: FT232RL-REEL, Downloads:SOP65P780X200-28N
- moved JP2 17.8 mm to (6.35, 50.8)
Connections:
- net N$1 renamed VINT
- net N$16 renamed TOSC1
- net N$18 renamed TOSC2
- net N$2 renamed VCP
- net N$4 renamed AREF
- net RESET renamed !RESET!
- new net 3V3: C11.1, U5.17
- new net N$2: B1.1, U5.20, U5.4
- new net N$4: J3.3, U5.15
- new net N$5: J3.2, U5.16
- new net VCC: B1.2, C13.+, J3.1
- net GND: now also C11.2, C13.-, J3.5, U5.18, U5.21, U5.25, U5.26, U5.7
- net RXD: now also U5.1
- net TXD: now also U5.5

Commit message: Add files via upload
Parts:
- added B2: (no value), ME507:0805
- added C14, C15: 22pF, rcl:C0805
- added C16: 4.7uF, rcl:A/3216-18W
- added C17: 100nF, rcl:C0805
- added R10, R11: 270, rcl:R0805
- added R2: 4.7k, rcl:R0805
- added R3: 330, rcl:R0805
- added R4, R5: (no value), rcl:R0805
- added R6: 100m, rcl:R0805
- added R7, R8, R9: 500, rcl:R0805
- added SW1: SW, ME507:B3F-10XX
- added Y2: 30MHz, Downloads:XTAL_ECS-160-20-3X-TR
- C6, C7: value 22pF -> 20pF
- R1: value 200m -> 400m
Connections:
- net N$4 renamed DP
- net N$5 renamed DM
- removed net !SLEEP!: U2.1
- removed net 3V3: C11.1, U5.17
- removed net N$2: B1.1, U5.20, U5.4
- removed net N$3: R1.1, U2.3, U2.6
- removed net VSS: U3.3
- new net +3V3: C11.1, JP4.4, R4.1, R5.1, U5.17
- new net AISEN: R6.1, U2.3
- new net AVCC: B2.1, C10.1, U1.18
- new net BISEN: R1.1, U2.6
- new net BUS0: R11.2, U5.23
- new net BUS1: R10.2, U5.22
- new net FCKI: C14.1, U3.2, Y2.1
- new net FCKO: C15.1, U3.1, Y2.2
- new net MI: R9.2, U3.6
- new net MO: R8.2, U3.7
- new net N$12: J3.4
- new net N$16: U5.27
- new net N$17: U5.28
- new net N$18: U5.19
- new net N$20: U5.9
- new net N$21: U5.6
- new net N$22: U5.10
- new net N$23: U5.2
- new net N$24: U5.13
- new net N$25: U5.14
- new net N$26: U5.12
- new net N$27: U3.10
- new net N$28: U3.9
- new net SCK: JP1.3, R7.1, U1.17
- new net SW: R3.1, SW1.1
- new net VCCIO: B1.1, C16.+, R10.1, R11.1, U5.20, U5.4
- net !RESET!: now also C17.1, R2.1, R3.2
- net !SS!: now also U1.32; no longer U1.17
- net +5V: now also B2.2, R2.2, U2.1; no longer C10.1, U1.18
- net AIN1: now also U1.9; no longer U1.1
- net AIN2: now also U1.10; no longer U1.9
- net BIN1: now also U1.13; no longer U1.10
- net BIN2: now also U1.14; no longer U1.13
- net ENCA: now also JP4.3, R4.2; no longer JP4.4
- net ENCB: now also JP4.2, R5.2; no longer JP4.3
- net GND: now also C14.2, C15.2, C16.-, C17.2, JP4.1, R6.2, SW1.3, U3.3
- net MISO: now also R9.1, U1.16; no longer U1.15, U3.6
- net MOSI: now also R8.1, U1.15; no longer U1.16, U3.7
- net SCLK: now also R7.2; no longer JP1.3, U1.14

Commit message: Add files via upload
Parts:
- added D1: HSMC-C190, HSMC-C190:LEDM1608X80
- added S1: 5-1437565-0, 5-1437565-0:SW_5-1437565-0
- C1, C10, C11, C12, C17, C2, C4, C5, C8, C9: device rcl:C0805 -> C2012X7R1V225K125AE:CAPC2112X150N
- C14, C15, C6, C7: device rcl:C0805 -> 101X15N220MV4E:CAPC2012X127N
- R1: device rcl:R0805 -> RL1206FR-070R4L:RESC3116X65N
