File: main.brd (EAGLE design)
At the start: 76.2 x 63.5 mm, 46 parts, among them J1 PJ-015AH-SMT-TR, J3 1734510-1, SW1 SW, U1 ATMEGA328P-AU, U2 DRV8833PWPR, U3 LS7366R-TS, U4 LP38691DTX-5.0/NOPB, U5 FT232RL-REEL, Y1 16MHz, Y2 30MHz

Commit message: Add files via upload
Parts:
- removed D1: HSMC-C190, HSMC-C190:LEDM1608X80
- removed SW1: SW, ME507:B3F-10XX
- C1, C10, C11, C12, C17, C2, C4, C5, C8, C9: device C2012X7R1V225K125AE:CAPC2112X150N -> rcl:C0805
- C14, C15: value 22pF -> 20pF; device 101X15N220MV4E:CAPC2012X127N -> rcl:C0805
- C6, C7: device 101X15N220MV4E:CAPC2012X127N -> rcl:C0805
- R1: device RL1206FR-070R4L:RESC3116X65N -> rcl:R0805
- S1: device 5-1437565-0:SW_5-1437565-0 -> Downloads:SW_5-1437565-0
- moved S1 152.8 mm to (6.35, 44.5), turned to 270 degrees
- moved C17 127.8 mm to (19.1, 41.9), turned to 270 degrees
- moved R11 120.4 mm to (19.1, 21.6), turned to 90 degrees
- moved R10 113.1 mm to (14.0, 21.6), turned to 90 degrees
- moved C15 110.9 mm to (27.9, 55.9), turned to 180 degrees
- moved R9 109.6 mm to (39.4, 21.6)
- moved R7 105.1 mm to (39.4, 26.7)
- moved R6 102.4 mm to (63.5, 11.4), turned to 270 degrees
- moved R8 100.7 mm to (39.4, 16.5)
- moved C14 100.2 mm to (27.9, 50.8), turned to 180 degrees
- moved Y2 97.7 mm to (35.6, 53.3), turned to 90 degrees
- moved R5 72.9 mm to (49.5, 12.7)
- moved C16 71.9 mm to (16.5, 14.0)
- moved R4 71.5 mm to (49.5, 16.5)
- moved R2 63.2 mm to (14.0, 47.0), turned to 90 degrees
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Connections:
- new net LFLAG: U1.2, U3.8
- new net N$2: U5.3
- new net N$3: U5.11
- new net N$4: U3.13
- net !FAULT!: now also U1.1
- net GND: now also S1.3, S1.4; no longer SW1.3
- net SW: now also S1.1, S1.2; no longer SW1.1

Commit message: Add files via upload
Parts:
- added D1: RED LED, HSMC-C190:LEDM1608X80
- added D2, D3: GREEN LED, HSMC-C190:LEDM1608X80
- added R14: 270, rcl:R0805
Connections:
- new net N$5: R14.2, U1.19
- new net N$6: D1.A, R14.1
- new net N$7: D3.A, R11.1
- net GND: now also D1.C, D2.C, D3.C
- net VCCIO: now also D2.A; no longer R11.1
Changed lines of the file:
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@@
 <drawing>
 <settings>
-<setting alwaysvectorfont="no"/>
+<setting alwaysvectorfont="yes"/>
 <setting verticaltext="up"/>
 </settings>
@@
 <attribute name="VALUE" x="1.44023125" y="50.011059375" size="1.27253125" layer="27" rot="R270"/>
 </element>
+<element name="R14" library="rcl" library_urn="urn:adsk.eagle:library:334" package="R0805" package3d_urn="urn:adsk.eagle:package:23553/2" value="270" x="0" y="-19.05" smashed="yes">
+<attribute name="NAME" x="-0.635" y="-17.78" size="1.27" layer="25"/>
+<attribute name="POPULARITY" value="85" x="0" y="-19.05" size="1.778" layer="27" display="off"/>
+<attribute name="SPICEPREFIX" value="R" x="0" y="-19.05" size="1.778" layer="27" display="off"/>
+<attribute name="VALUE" x="-0.635" y="-21.59" size="1.27" layer="27"/>
+</element>
+<element name="D1" library="HSMC-C190" package="LEDM1608X80" value="RED LED" x="0" y="-21.59" smashed="yes">
+<attribute name="DESCRIPTION" value=" LED; SMD; 0603; red; 28.5-90mcd; 1.6x0.8x0.8mm; 170°; 1.9÷2.4V; 20mA " x="0" y="-21.59" size="1.778" layer="27" display="off"/>
+<attribute name="DIGI-KEY_PART_NUMBER" value="516-1421-1-ND" x="0" y="-21.59" size="1.778" layer="27" display="off"/>
+<attribute name="DIGI-KEY_PURCHASE_URL" value="https://www.digikey.com/product-detail/en/broadcom-limited/HSMC-C190/516-1421-1-ND/637745?utm_source=snapeda&amp;utm_medium=aggregator&amp;utm_campaign=symbol" x="0" y="-21.59" size="1.778" layer="27" display="off"/>
+<attribute name="MF" value="Broadcom Limited" x="0" y="-21.59" size="1.778" layer="27" display="off"/>
+<attribute name="MP" value="HSMC-C190" x="0" y="-21.59" size="1.778" layer="27" display="off"/>
+<attribute name="NAME" x="-1.52" y="-20.905" size="0.4064" layer="25"/>
+<attribute name="PACKAGE" value="0603 Broadcom" x="0" y="-21.59" size="1.778" layer="27" display="off"/>
+<attribute name="VALUE" x="-1.52" y="-22.695" size="0.4064" layer="27"/>
+</element>
+<element name="D2" library="HSMC-C190" package="LEDM1608X80" value="GREEN LED" x="0" y="-25.4" smashed="yes">
+<attribute name="DESCRIPTION" value=" LED; SMD; 0603; red; 28.5-90mcd; 1.6x0.8x0.8mm; 170°; 1.9÷2.4V; 20mA " x="0" y="-25.4" size="1.778" layer="27" display="off"/>
+<attribute name="DIGI-KEY_PART_NUMBER" value="516-1421-1-ND" x="0" y="-25.4" size="1.778" layer="27" display="off"/>
+<attribute name="DIGI-KEY_PURCHASE_URL" value="https://www.digikey.com/product-detail/en/broadcom-limited/HSMC-C190/516-1421-1-ND/637745?utm_source=snapeda&amp;utm_medium=aggregator&amp;utm_campaign=symbol" x="0" y="-25.4" size="1.778" layer="27" display="off"/>
+<attribute name="MF" value="Broadcom Limited" x="0" y="-25.4" size="1.778" layer="27" display="off"/>
+<attribute name="MP" value="HSMC-C190" x="0" y="-25.4" size="1.778" layer="27" display="off"/>
+<attribute name="NAME" x="-1.52" y="-24.715" size="0.4064" layer="25"/>
+<attribute name="PACKAGE" value="0603 Broadcom" x="0" y="-25.4" size="1.778" layer="27" display="off"/>
+<attribute name="VALUE" x="-1.52" y="-26.505" size="0.4064" layer="27"/>
+</element>
+<element name="D3" library="HSMC-C190" package="LEDM1608X80" value="GREEN LED" x="0" y="-29.21" smashed="yes">
+<attribute name="DESCRIPTION" value=" LED; SMD; 0603; red; 28.5-90mcd; 1.6x0.8x0.8mm; 170°; 1.9÷2.4V; 20mA " x="0" y="-29.21" size="1.778" layer="27" display="off"/>
+<attribute name="DIGI-KEY_PART_NUMBER" value="516-1421-1-ND" x="0" y="-29.21" size="1.778" layer="27" display="off"/>
+<attribute name="DIGI-KEY_PURCHASE_URL" value="https://www.digikey.com/product-detail/en/broadcom-limited/HSMC-C190/516-1421-1-ND/637745?utm_source=snapeda&amp;utm_medium=aggregator&amp;utm_campaign=symbol" x="0" y="-29.21" size="1.778" layer="27" display="off"/>
+<attribute name="MF" value="Broadcom Limited" x="0" y="-29.21" size="1.778" layer="27" display="off"/>
+<attribute name="MP" value="HSMC-C190" x="0" y="-29.21" size="1.778" layer="27" display="off"/>
+<attribute name="NAME" x="-1.52" y="-28.525" size="0.4064" layer="25"/>
+<attribute name="PACKAGE" value="0603 Broadcom" x="0" y="-29.21" size="1.778" layer="27" display="off"/>
+<attribute name="VALUE" x="-1.52" y="-30.315" size="0.4064" layer="27"/>
+</element>
 </elements>
 <signals>
@@
 <contactref element="S1" pad="3"/>
 <contactref element="S1" pad="4"/>
+<contactref element="D1" pad="C"/>
+<contactref element="D3" pad="C"/>
+<contactref element="D2" pad="C"/>
+<wire x1="62.395" y1="59.56" x2="67.145" y2="59.56" width="0" layer="19" extent="1-1"/>
+<wire x1="46.99" y1="55.88" x2="62.395" y2="59.56" width="0" layer="19" extent="1-1"/>
+<wire x1="49.53" y1="40.96" x2="46.99" y2="55.88" width="0" layer="19" extent="1-1"/>
+<wire x1="43.18" y1="40.96" x2="49.53" y2="40.96" width="0" layer="19" extent="1-1"/>
+<wire x1="42.855" y1="33.67" x2="43.18" y2="40.96" width="0" layer="19" extent="1-1"/>
+<wire x1="54.45" y1="31.75" x2="49.53" y2="40.96" width="0" layer="19" extent="1-1"/>
+<wire x1="64.77" y1="30.16" x2="54.45" y2="31.75" width="0" layer="19" extent="1-1"/>
+<wire x1="65.715003125" y1="23.1394" x2="64.77" y2="30.16" width="0" layer="19" extent="1-1"/>
+<wire x1="66.04" y1="20.32" x2="65.715003125" y2="23.1394" width="0" layer="19" extent="1-1"/>
+<wire x1="68.58" y1="10.48" x2="66.04" y2="20.32" width="0" layer="19" extent="1-1"/>
+<wire x1="63.5" y1="10.48" x2="68.58" y2="10.48" width="0" layer="19" extent="1-1"/>
+<wire x1="57.15" y1="11.43" x2="63.5" y2="10.48" width="0" layer="19" extent="1-1"/>
+<wire x1="31.75" y1="42.86" x2="43.18" y2="40.96" width="0" layer="19" extent="1-1"/>
+<wire x1="25.4" y1="42.86" x2="31.75" y2="42.86" width="0" layer="19" extent="1-1"/>
+<wire x1="19.05" y1="40.96" x2="25.4" y2="42.86" width="0" layer="19" extent="1-1"/>
+<wire x1="27.54" y1="36.05" x2="25.4" y2="42.86" width="0" layer="19" extent="1-1"/>
+<wire x1="26.99" y1="50.8" x2="25.4" y2="42.86" width="0" layer="19" extent="1-1"/>
+<wire x1="26.99" y1="55.88" x2="26.99" y2="50.8" width="0" layer="19" extent="1-1"/>
+<wire x1="28.34" y1="27.45" x2="27.54" y2="36.05" width="0" layer="19" extent="1-1"/>
+<wire x1="26.74" y1="27.45" x2="28.34" y2="27.45" width="0" layer="19" extent="1-1"/>
+<wire x1="25.4" y1="20.64" x2="26.74" y2="27.45" width="0" layer="19" extent="1-1"/>
+<wire x1="31.75" y1="20.64" x2="25.4" y2="20.64" width="0" layer="19" extent="1-1"/>
+<wire x1="11.755" y1="35.375" x2="19.05" y2="40.96" width="0" layer="19" extent="1-1"/>
+<wire x1="11.105" y1="28.125" x2="11.755" y2="35.375" width="0" layer="19" extent="1-1"/>
+<wire x1="9.155" y1="28.125" x2="11.105" y2="28.125" width="0" layer="19" extent="1-1"/>
+<wire x1="13.705" y1="28.125" x2="11.105" y2="28.125" width="0" layer="19" extent="1-1"/>
+<wire x1="14.355" y1="28.125" x2="13.705" y2="28.125" width="0" layer="19" extent="1-1"/>
+<wire x1="4.1" y1="39.9" x2="11.755" y2="35.375" width="0" layer="19" extent="1-1"/>
+<wire x1="4.1" y1="49" x2="4.1" y2="39.9" width="0" layer="19" extent="1-1"/>
+<wire x1="3.81" y1="20.64" x2="9.155" y2="28.125" width="0" layer="19" extent="1-1"/>
+<wire x1="10.365" y1="13.97" x2="3.81" y2="20.64" width="0" layer="19" extent="1-1"/>
+<wire x1="15.035" y1="13.97" x2="10.365" y2="13.97" width="0" layer="19" extent="1-1"/>
+<wire x1="14.3" y1="7.59" x2="15.035" y2="13.97" width="0" layer="19" extent="1-1"/>
+<wire x1="16.51" y1="58.42" x2="26.99" y2="55.88" width="0" layer="19" extent="1-1"/>
+<wire x1="26.67" y1="5.4" x2="14.3" y2="7.59" width="0" layer="19" extent="1-1"/>
+<wire x1="33.02" y1="5.4" x2="26.67" y2="5.4" width="0" layer="19" extent="1-1"/>
+<wire x1="45.72" y1="5.08" x2="33.02" y2="5.4" width="0" layer="19" extent="1-1"/>
+<wire x1="-0.75" y1="-21.59" x2="14.3" y2="7.59" width="0" layer="19" extent="1-1"/>
+<wire x1="-0.75" y1="-25.4" x2="-0.75" y2="-21.59" width="0" layer="19" extent="1-1"/>
+<wire x1="-0.75" y1="-29.21" x2="-0.75" y2="-25.4" width="0" layer="19" extent="1-1"/>
 </signal>
 <signal name="BISEN">
@@
 <contactref element="C16" pad="+"/>
 <contactref element="R10" pad="1"/>
-<contactref element="R11" pad="1"/>
+<contactref element="D2" pad="A"/>
 <wire x1="10.455" y1="28.125" x2="13.705" y2="35.375" width="0" layer="19" extent="1-1"/>
 <wire x1="8.89" y1="22.59" x2="10.455" y2="28.125" width="0" layer="19" extent="1-1"/>
 <wire x1="13.97" y1="20.64" x2="8.89" y2="22.59" width="0" layer="19" extent="1-1"/>
-<wire x1="19.05" y1="20.64" x2="13.97" y2="20.64" width="0" layer="19" extent="1-1"/>
-<wire x1="17.985" y1="13.97" x2="19.05" y2="20.64" width="0" layer="19" extent="1-1"/>
+<wire x1="17.985" y1="13.97" x2="13.97" y2="20.64" width="0" layer="19" extent="1-1"/>
+<wire x1="0.75" y1="-25.4" x2="17.985" y2="13.97" width="0" layer="19" extent="1-1"/>
 </signal>
 <signal name="VCC">
@@
 <wire x1="25.94" y1="27.45" x2="48.585" y2="31.07" width="0" layer="19" extent="1-1"/>
 </signal>
+<signal name="N$5">
+<contactref element="U1" pad="19"/>
+<contactref element="R14" pad="2"/>
+<wire x1="0.95" y1="-19.05" x2="29.14" y2="36.05" width="0" layer="19" extent="1-1"/>
+</signal>
+<signal name="N$6">
+<contactref element="R14" pad="1"/>
+<contactref element="D1" pad="A"/>
+<wire x1="-0.95" y1="-19.05" x2="0.75" y2="-21.59" width="0" layer="19" extent="1-1"/>
+</signal>
+<signal name="N$7">
+<contactref element="R11" pad="1"/>
+<contactref element="D3" pad="A"/>
+<wire x1="0.75" y1="-29.21" x2="19.05" y2="20.64" width="0" layer="19" extent="1-1"/>
+</signal>
 </signals>

Commit message: Add files via upload
Parts:
- C16: device rcl:A/3216-18W -> rcl:E5-5
- C3: device rcl:153CLV-0605 -> rcl:E5-4
Changed lines of the file:
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@@
 <attribute name="VALUE" x="66.04" y="12.065" size="1.27" layer="27" rot="R270"/>
 </element>
-<element name="C3" library="rcl" library_urn="urn:adsk.eagle:library:334" package="153CLV-0605" package3d_urn="urn:adsk.eagle:package:23398/2" value="10uF" x="57.15" y="31.75" smashed="yes">
+<element name="C3" library="rcl" library_urn="urn:adsk.eagle:library:334" package="E5-4" package3d_urn="urn:adsk.eagle:package:23370/1" value="10uF" x="57.15" y="31.75" smashed="yes">
 <attribute name="NAME" x="53.76" y="35.38" size="1.27" layer="25"/>
-<attribute name="POPULARITY" value="8" x="57.15" y="31.75" size="1.778" layer="27" display="off"/>
+<attribute name="POPULARITY" value="0" x="57.15" y="31.75" size="1.778" layer="27" display="off"/>
 <attribute name="SPICEPREFIX" value="C" x="57.15" y="31.75" size="1.778" layer="27" display="off"/>
 <attribute name="VALUE" x="53.725" y="26.865" size="1.27" layer="27"/>
@@
 <attribute name="VALUE" x="29.21" y="58.42" size="1.27" layer="27" rot="R180"/>
 </element>
-<element name="C16" library="rcl" library_urn="urn:adsk.eagle:library:334" package="A/3216-18W" package3d_urn="urn:adsk.eagle:package:23408/2" value="4.7uF" x="16.51" y="13.97" smashed="yes">
+<element name="C16" library="rcl" library_urn="urn:adsk.eagle:library:334" package="E5-5" package3d_urn="urn:adsk.eagle:package:23367/2" value="4.7uF" x="16.51" y="13.97" smashed="yes">
 <attribute name="NAME" x="14.56" y="14.97" size="1.27" layer="25"/>
-<attribute name="POPULARITY" value="1" x="16.51" y="13.97" size="1.778" layer="27" display="off"/>
+<attribute name="POPULARITY" value="5" x="16.51" y="13.97" size="1.778" layer="27" display="off"/>
 <attribute name="SPICEPREFIX" value="C" x="16.51" y="13.97" size="1.778" layer="27" display="off"/>
 <attribute name="VALUE" x="14.56" y="11.645" size="1.27" layer="27"/>
@@
 <wire x1="43.18" y1="40.96" x2="49.53" y2="40.96" width="0" layer="19" extent="1-1"/>
 <wire x1="42.855" y1="33.67" x2="43.18" y2="40.96" width="0" layer="19" extent="1-1"/>
-<wire x1="54.45" y1="31.75" x2="49.53" y2="40.96" width="0" layer="19" extent="1-1"/>
-<wire x1="64.77" y1="30.16" x2="54.45" y2="31.75" width="0" layer="19" extent="1-1"/>
-<wire x1="65.715003125" y1="23.1394" x2="64.77" y2="30.16" width="0" layer="19" extent="1-1"/>
-<wire x1="66.04" y1="20.32" x2="65.715003125" y2="23.1394" width="0" layer="19" extent="1-1"/>
-<wire x1="68.58" y1="10.48" x2="66.04" y2="20.32" width="0" layer="19" extent="1-1"/>
-<wire x1="63.5" y1="10.48" x2="68.58" y2="10.48" width="0" layer="19" extent="1-1"/>
-<wire x1="57.15" y1="11.43" x2="63.5" y2="10.48" width="0" layer="19" extent="1-1"/>
 <wire x1="31.75" y1="42.86" x2="43.18" y2="40.96" width="0" layer="19" extent="1-1"/>
 <wire x1="25.4" y1="42.86" x2="31.75" y2="42.86" width="0" layer="19" extent="1-1"/>
@@
 <wire x1="4.1" y1="39.9" x2="11.755" y2="35.375" width="0" layer="19" extent="1-1"/>
 <wire x1="4.1" y1="49" x2="4.1" y2="39.9" width="0" layer="19" extent="1-1"/>
+<wire x1="19.05" y1="13.97" x2="25.4" y2="20.64" width="0" layer="19" extent="1-1"/>
+<wire x1="14.3" y1="7.59" x2="19.05" y2="13.97" width="0" layer="19" extent="1-1"/>
+<wire x1="10.365" y1="13.97" x2="14.3" y2="7.59" width="0" layer="19" extent="1-1"/>
 <wire x1="3.81" y1="20.64" x2="9.155" y2="28.125" width="0" layer="19" extent="1-1"/>
-<wire x1="10.365" y1="13.97" x2="3.81" y2="20.64" width="0" layer="19" extent="1-1"/>
-<wire x1="15.035" y1="13.97" x2="10.365" y2="13.97" width="0" layer="19" extent="1-1"/>
-<wire x1="14.3" y1="7.59" x2="15.035" y2="13.97" width="0" layer="19" extent="1-1"/>
 <wire x1="16.51" y1="58.42" x2="26.99" y2="55.88" width="0" layer="19" extent="1-1"/>
-<wire x1="26.67" y1="5.4" x2="14.3" y2="7.59" width="0" layer="19" extent="1-1"/>
+<wire x1="26.67" y1="5.4" x2="19.05" y2="13.97" width="0" layer="19" extent="1-1"/>
 <wire x1="33.02" y1="5.4" x2="26.67" y2="5.4" width="0" layer="19" extent="1-1"/>
 <wire x1="45.72" y1="5.08" x2="33.02" y2="5.4" width="0" layer="19" extent="1-1"/>
+<wire x1="57.15" y1="11.43" x2="45.72" y2="5.08" width="0" layer="19" extent="1-1"/>
+<wire x1="63.5" y1="10.48" x2="57.15" y2="11.43" width="0" layer="19" extent="1-1"/>
+<wire x1="68.58" y1="10.48" x2="63.5" y2="10.48" width="0" layer="19" extent="1-1"/>
+<wire x1="66.04" y1="20.32" x2="63.5" y2="10.48" width="0" layer="19" extent="1-1"/>
+<wire x1="65.715003125" y1="23.1394" x2="66.04" y2="20.32" width="0" layer="19" extent="1-1"/>
+<wire x1="64.77" y1="30.16" x2="65.715003125" y2="23.1394" width="0" layer="19" extent="1-1"/>
+<wire x1="59.69" y1="31.75" x2="64.77" y2="30.16" width="0" layer="19" extent="1-1"/>
 <wire x1="-0.75" y1="-21.59" x2="14.3" y2="7.59" width="0" layer="19" extent="1-1"/>
 <wire x1="-0.75" y1="-25.4" x2="-0.75" y2="-21.59" width="0" layer="19" extent="1-1"/>
@@
 <contactref element="C2" pad="1"/>
 <contactref element="C3" pad="+"/>
-<wire x1="59.85" y1="31.75" x2="64.77" y2="40.66" width="0" layer="19" extent="1-1"/>
-<wire x1="66.365" y1="23.1394" x2="59.85" y2="31.75" width="0" layer="19" extent="1-1"/>
-<wire x1="71.12" y1="30.16" x2="66.365" y2="23.1394" width="0" layer="19" extent="1-1"/>
-<wire x1="49.53" y1="42.86" x2="59.85" y2="31.75" width="0" layer="19" extent="1-1"/>
+<wire x1="71.12" y1="30.16" x2="64.77" y2="40.66" width="0" layer="19" extent="1-1"/>
+<wire x1="66.365" y1="23.1394" x2="71.12" y2="30.16" width="0" layer="19" extent="1-1"/>
+<wire x1="54.61" y1="31.75" x2="64.77" y2="40.66" width="0" layer="19" extent="1-1"/>
+<wire x1="49.53" y1="42.86" x2="54.61" y2="31.75" width="0" layer="19" extent="1-1"/>
 <wire x1="49.275" y1="49.3776" x2="49.53" y2="42.86" width="0" layer="19" extent="1-1"/>
 </signal>
@@
 <wire x1="8.89" y1="22.59" x2="10.455" y2="28.125" width="0" layer="19" extent="1-1"/>
 <wire x1="13.97" y1="20.64" x2="8.89" y2="22.59" width="0" layer="19" extent="1-1"/>
-<wire x1="17.985" y1="13.97" x2="13.97" y2="20.64" width="0" layer="19" extent="1-1"/>
-<wire x1="0.75" y1="-25.4" x2="17.985" y2="13.97" width="0" layer="19" extent="1-1"/>
+<wire x1="13.97" y1="13.97" x2="13.97" y2="20.64" width="0" layer="19" extent="1-1"/>
+<wire x1="0.75" y1="-25.4" x2="13.97" y2="13.97" width="0" layer="19" extent="1-1"/>
 </signal>
 <signal name="VCC">

Commit message: Add files via upload
Parts:
- moved D1 56.6 mm to (39.4, 19.1), turned to 180 degrees
- moved R14 51.4 mm to (39.4, 14.0), turned to 90 degrees
- moved D3 49.5 mm to (19.1, 16.5), turned to 270 degrees
- moved D2 44.2 mm to (14.0, 16.5), turned to 270 degrees
- moved R7 10.2 mm to (39.4, 36.8)
- moved S1 9.25 mm to (8.89, 53.3)
- moved JP2 8.98 mm to (21.6, 55.9)
- moved R9 8.89 mm to (39.4, 30.5)
- moved R3 7.62 mm to (6.35, 41.9), turned to 270 degrees
- moved R8 7.62 mm to (39.4, 24.1)
- moved C16 6.35 mm to (20.3, 8.89), turned to 270 degrees
- moved R2 5.24 mm to (12.7, 41.9)
- moved C15 5.24 mm to (33.0, 57.1)
- moved C14 5.08 mm to (33.0, 50.8)
- moved C3 3.81 mm to (57.1, 35.6), turned to 270 degrees
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Connections:
- net DM renamed N$9
- net DP renamed N$10
- removed net N$7: D3.A, R11.1
- new net RXLED: D2.C, R10.1
- new net TXLED: D3.C, R11.1
- net FLOW: now also U1.12
- net GND: now also R14.1; no longer D1.C, D2.C, D3.C
- net N$5: now also D1.A, U1.11; no longer R14.2, U1.19
- net N$6: now also D1.C, R14.2; no longer D1.A, R14.1
- net VCCIO: now also D3.A; no longer R10.1
Routing:
- net +5V: track 0.00 -> 161.5 mm, vias 0 -> 2
- net +3V3: track 0.00 -> 73.8 mm, vias 0 -> 2
- net !RESET!: track 0.00 -> 72.6 mm, vias 0 -> 2
- net !FAULT!: track 0.00 -> 63.5 mm, vias 0 -> 2
- net BIN2: track 0.00 -> 50.3 mm, vias 0 -> 2
- net BIN1: track 0.00 -> 48.3 mm, vias 0 -> 2
- net VIN: track 0.00 -> 45.4 mm
- net SCK: track 0.00 -> 44.3 mm, vias 0 -> 4
- net AIN2: track 0.00 -> 40.6 mm, vias 0 -> 2
- net MISO: track 0.00 -> 40.1 mm, vias 0 -> 2
- net AIN1: track 0.00 -> 37.8 mm, vias 0 -> 2
- net MOSI: track 0.00 -> 36.3 mm
- net VCCIO: track 0.00 -> 34.9 mm
- net N$9: track 0.00 -> 31.6 mm
- net FCKO: track 0.00 -> 29.6 mm, vias 0 -> 2
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
Commit message: Add files via upload
Parts:
- added R12: 1M, rcl:R0805
- C13: device rcl:A/3216-18W -> rcl:C0805
- JP2: device pinhead:2X04 -> Downloads:2X04
- JP3, JP4: device pinhead:1X04 -> Downloads:1X04
- moved JP1 49.9 mm to (36.8, 55.2)
- moved Y2 41.2 mm to (56.5, 15.9), turned to 0 degrees
- moved C15 40.0 mm to (59.7, 27.3), turned to 90 degrees
- moved C14 30.7 mm to (52.7, 27.3), turned to 90 degrees
- moved R14 17.1 mm to (45.7, 29.8)
- moved JP4 14.4 mm to (47.0, 5.08), turned to 180 degrees
- moved U3 13.5 mm to (43.8, 20.3), turned to 270 degrees
- moved R7 12.7 mm to (52.1, 36.2), turned to 270 degrees
- moved R8 12.1 mm to (39.4, 36.2), turned to 270 degrees
- moved D1 10.8 mm to (39.4, 29.8), turned to 270 degrees
- moved R4 8.98 mm to (50.8, 10.2), turned to 180 degrees
- moved R9 8.54 mm to (45.7, 36.2), turned to 270 degrees
- moved R5 7.41 mm to (43.2, 10.2)
- moved C3 1.80 mm to (58.4, 34.3)
- moved Y1 1.42 mm to (31.1, 12.7)
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Connections:
- removed net ENCA: JP4.3, R4.2, U3.12
- removed net ENCB: JP4.2, R5.2, U3.11
- new net N$7: JP4.3, R5.2, U3.11
- new net N$8: JP4.2, R4.2, U3.12
- net FCKI: now also R12.2
- net FCKO: now also R12.1
- net GND: now also C13.2; no longer C13.-
- net VCC: now also C13.1; no longer C13.+
Routing:
- net ENCB: track 29.5 -> 0.00 mm, vias 2 -> 0
- net ENCA: track 26.0 -> 0.00 mm, vias 2 -> 0
- net !RESET!: track 72.6 -> 50.3 mm
- net N$8: track 0.00 -> 15.3 mm
- net N$7: track 0.00 -> 13.2 mm
- net MO: track 9.99 -> 23.0 mm
- net MI: track 5.59 -> 18.3 mm
- net SCLK: track 7.48 -> 17.2 mm
- net !FAULT!: track 63.5 -> 54.5 mm
- net MOSI: track 36.3 -> 27.3 mm, vias 0 -> 2
- net LFLAG: track 29.2 -> 20.8 mm
- net +5V: track 161.5 -> 153.6 mm, vias 2 -> 4
- net N$5: track 15.3 -> 7.73 mm
- net N$9: track 31.6 -> 25.8 mm, vias 0 -> 1
- net FCKO: track 29.6 -> 24.3 mm
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Other:
- outline, holes or cut-outs redrawn
