File: main.brd (EAGLE design)
At the start: 76.2 x 63.5 mm, 49 parts, among them J1 PJ-015AH-SMT-TR, J3 1734510-1, U1 ATMEGA328P-AU, U2 DRV8833PWPR, U3 LS7366R-TS, U4 LP38691DTX-5.0/NOPB, U5 FT232RL-REEL, Y1 16MHz, Y2 30MHz

Commit message: Add files via upload
Parts:
- B1, B2: value (none) -> 100
- J1: value PJ-015AH-SMT-TR -> PJ-036AH-SMT-TR; device Downloads:CUI_PJ-015AH-SMT-TR -> Downloads:CUI_PJ-036AH-SMT-TR
- R4, R5: value (none) -> 4.7
- U3: value LS7366R-TS -> LS7366R-S; device Downloads:SOP65P640X110-14N -> Downloads:SOIC127P600X175-14N
- moved J1 3.86 mm to (60.3, 47.6)
- moved J3 0.64 mm to (10.8, 1.91)
Connections:
- net N$10 renamed DP
- net N$5 renamed PD7
- net N$6 renamed LED
- net N$7 renamed ENCB
- net N$8 renamed ENCA
- net N$9 renamed DM
Routing:
- net VIN: track 46.5 -> 53.7 mm
- net MO: track 23.0 -> 25.2 mm
- net LFLAG: track 20.8 -> 18.9 mm
- net FCKO: track 24.3 -> 22.6 mm
- net MI: track 18.3 -> 19.8 mm
- net FCKI: track 21.9 -> 20.6 mm
- net SCLK: track 17.2 -> 18.2 mm
- net +5V: track 153.6 -> 154.3 mm
- net DP: track 23.3 -> 23.9 mm
- net VCC: track 14.4 -> 15.1 mm
- net AOUT2: track 16.0 -> 16.4 mm, vias 0 -> 1
- net BOUT2: vias 0 -> 1
- added copper zone on layer 1, net +5V
- added copper zone on layer 1, net AOUT1
- added copper zone on layer 16, net AOUT2
- added copper zone on layer 1, net BOUT1
- added copper zone on layer 16, net BOUT2
- added copper zone on layer 1, net VIN
Other:
- board text added: "+3V3"
- board text added: "+5V"
- board text added: "A"
- board text added: "A1"
- board text added: "A2"
- board text added: "ADC"
- board text added: "B"
- board text added: "B1"
- board text added: "B2"
- board text added: "FLOW"
- board text added: "GND"
- board text added: "Josh Castle Kylie Fernandez ME-507 2019 Plantiful Care"
- board text added: "MISO"
- board text added: "MOSI"
- board text added: "RST"
- board text added: "SCK"
- board text added: "SCL"
- board text added: "SDA"

Commit message: Add files via upload
Parts:
- moved U4 7.43 mm to (56.5, 53.3), turned to 270 degrees
- moved JP1 3.17 mm to (36.8, 52.1)
- moved JP2 1.90 mm to (22.2, 53.3)
- moved S1 1.42 mm to (9.53, 52.1)
- moved J1 1.27 mm to (60.3, 46.4)
- moved C3 0.90 mm to (59.1, 34.9)
- moved C4 0.63 mm to (45.7, 42.5)
- moved C5 0.63 mm to (52.1, 42.5)
Routing:
- net +5V: track 154.3 -> 150.0 mm, vias 4 -> 8
- net MOSI: track 27.3 -> 24.2 mm
- net SCK: track 42.2 -> 39.0 mm
- net MISO: track 40.4 -> 37.2 mm
- net FLOW: track 28.0 -> 25.6 mm
- net SDA: track 23.5 -> 21.6 mm
- net SCL: track 25.4 -> 23.5 mm
- net ADC: track 21.8 -> 19.9 mm
- net !RESET!: track 50.3 -> 48.7 mm
- net FCKO: track 22.6 -> 23.8 mm
- net !FAULT!: track 54.5 -> 55.4 mm
- net VIN: track 53.7 -> 54.0 mm, vias 0 -> 5
- added copper zone on layer 16, net +5V
- added copper zone on layer 16, net VIN
Other:
- board size 76.2 x 63.5 mm -> 76.2 x 60.3 mm
