File: main.brd (EAGLE design)
At the start: 76.2 x 60.3 mm, 49 parts, among them J1 PJ-036AH-SMT-TR, J3 1734510-1, U1 ATMEGA328P-AU, U2 DRV8833PWPR, U3 LS7366R-S, U4 LP38691DTX-5.0/NOPB, U5 FT232RL-REEL, Y1 16MHz, Y2 30MHz

Commit message: Add files via upload
Parts:
- B2: value 100 -> 120
- R4, R5: value 4.7 -> 4.7k
