File: main.sch (EAGLE design)
At the start: 2 parts, among them U1 ATMEGA328P-AU, U2 DRV8833PWPR

Commit message: Add files via upload
Parts:
- added C1, C2: (no value), rcl:C-USC0805
- added C3: (no value), rcl:CPOL-US153CLV-0605
- added R1: 0.2, rcl:R-US_R0805
Connections:
- new net GND: C1.2, C3.-, R1.2, U1.GND, U2.EPAD, U2.GND
- new net N$1: C1.1, U2.VINT
- new net N$10: U2.!FAULT!
- new net N$11: U2.AOUT1
- new net N$12: U2.AOUT2
- new net N$13: U2.BOUT2
- new net N$14: U2.BOUT1
- new net N$2: C2.2, U2.VCP
- new net N$3: R1.1, U2.AISEN, U2.BISEN
- new net N$4: C2.1, C3.+, U2.VM
- new net N$5: U2.BIN1
- new net N$6: U2.BIN2
- new net N$7: U2.AIN2
- new net N$8: U2.AIN1
- new net N$9: U2.!SLEEP!
Other:
- moved on the sheet: U2

Commit message: Add files via upload
Parts:
- added U3: LP2985IM5-5.0, LP2985IM5-5.0:LP2985IM5-5.0
Changed lines of the file:
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@@
 <drawing>
 <settings>
-<setting alwaysvectorfont="no"/>
+<setting alwaysvectorfont="yes"/>
 <setting verticaltext="up"/>
 </settings>
@@
 <part name="GND4" library="supply1" library_urn="urn:adsk.eagle:library:371" deviceset="GND" device=""/>
 <part name="U2" library="Downloads" deviceset="DRV8833PWPR" device=""/>
+<part name="U3" library="LP2985IM5-5.0" deviceset="LP2985IM5-5.0" device=""/>
 </parts>
 <sheets>
@@
 <attribute name="VALUE" x="137.16" y="81.28" size="1.778" layer="96"/>
 </instance>
+<instance part="U3" gate="A" x="203.2" y="68.58" smashed="yes">
+<attribute name="NAME" x="197.73258125" y="77.48045" size="2.08525" layer="95" ratio="10" rot="SR0"/>
+<attribute name="VALUE" x="198.57055" y="50.5709" size="2.0858" layer="96" ratio="10" rot="SR0"/>
+</instance>
 </instances>

Commit message: Add files via upload
Parts:
- added C10, C11, C8, C9: 100nF, rcl:C-USC0805
- added C4, C5: 1uF, rcl:C-USC0805
- added C6, C7: 20pF, rcl:C-USC0805
- added J1: PJ-015AH-SMT-TR, Downloads:PJ-015AH-SMT-TR
- added JP1: (no value), pinhead:PINHD-2X3
- added U4: LP38691DTX-5.0/NOPB, Downloads:LP38691DTX-5.0/NOPB
- added Y1: 16MHz, Downloads:ECS-160-20-3X-TR
- C1: value (none) -> 2.2uF
- C2: value (none) -> 10nF
- C3: value (none) -> 10uF
- R1: value 0.2 -> 200m
- U3: value LP2985IM5-5.0 -> LS7366R-TS; device LP2985IM5-5.0:LP2985IM5-5.0 -> Downloads:LS7366R-TS
Connections:
- net N$10 renamed !FAULT!
- net N$11 renamed AOUT1
- net N$12 renamed AOUT2
- net N$13 renamed BOUT2
- net N$14 renamed BOUT1
- net N$5 renamed BIN1
- net N$6 renamed BIN2
- net N$7 renamed AIN2
- net N$8 renamed AIN1
- net N$9 renamed !SLEEP!
- new net !SS!: JP1.5, U1.PB5, U3.SS/
- new net +5V: C10.1, C11.1, C4.1, C8.1, C9.1, JP1.2, U1.AREF, U1.AVCC, U1.VCC, U3.VDD, U4.VOUT
- new net ADC: U1.PC3
- new net MISO: JP1.1, U1.PB3, U3.MISO
- new net MOSI: JP1.4, U1.PB4, U3.MOSI
- new net N$16: C7.1, U1.PB6, Y1.2
- new net N$18: C6.1, U1.PB7, Y1.1
- new net RXD: U1.PD0
- new net SCL: U1.PC5
- new net SCLK: JP1.3, U1.PB2, U3.SCK
- new net SDA: U1.PC4
- new net TXD: U1.PD1
- new net VIN: C5.1, J1.1, U4.VIN
- net GND: now also C10.2, C11.2, C4.2, C5.2, C6.2, C7.2, C8.2, C9.2, J1.2, J1.3, JP1.6, U4.GND
Other:
- note added: "AVR ISP Header"
- note added: "VCC Decoupling Capacitors"
- note added: "Voltage Regulator"
- moved on the sheet: C1, C2, C3, R1, U1, U2

Commit message: Add files via upload
Parts:
- removed C11: 100nF, rcl:C-USC0805
- added C12: 100nF, rcl:C-USC0805
- added JP2: (no value), pinhead:PINHD-2X4
- added JP3, JP4: (no value), pinhead:PINHD-1X4
- C6, C7: value 20pF -> 22pF
Connections:
- new net ENCA: JP4.4, U3.A
- new net ENCB: JP4.3, U3.B
- new net FLOW: JP2.7
- new net RESET: JP1.5, U1.PC6/!RESET
- net !SS!: no longer JP1.5
- net +5V: now also JP2.2, JP2.4, JP2.6; no longer C11.1, U1.AREF
- net ADC: now also JP2.5
- net AIN1: now also U1.PD3
- net AIN2: now also U1.PD5
- net AOUT1: now also JP3.4
- net AOUT2: now also JP3.3
- net BIN1: now also U1.PD6
- net BIN2: now also U1.PB1
- net BOUT1: now also JP3.1
- net BOUT2: now also JP3.2
- net GND: now also C12.2, JP2.8; no longer C11.2
- net N$4: now also C12.1, U1.AREF; no longer C2.1, C3.+, U2.VM
- net SCL: now also JP2.1
- net SDA: now also JP2.3
- net VIN: now also C2.1, C3.+, U2.VM
Other:
- note added: "Motor Driver"
- note added: "Quadrature Decoder"
- moved on the sheet: C10, C4, C5, C6, C7, C8, C9, J1, JP1, U3, U4, Y1

Commit message: Add files via upload
Parts:
- added B1: (no value), ME507:BEAD0805
- added C11: 100nF, rcl:C-USC0805
- added C13: 10nF, rcl:CPOL-USA/3216-18W
- added J3: 1734510-1, Downloads:1734510-1
- added U5: FT232RL-REEL, Downloads:FT232RL-REEL
Connections:
- net N$1 renamed VINT
- net N$16 renamed TOSC1
- net N$18 renamed TOSC2
- net N$2 renamed VCP
- net N$4 renamed AREF
- net RESET renamed !RESET!
- new net 3V3: C11.1, U5.3V3OUT
- new net N$2: B1.1, U5.VCC, U5.VCCIO
- new net N$4: J3.D+, U5.USBDP
- new net N$5: J3.D-, U5.USBDM
- new net VCC: B1.2, C13.+, J3.VCC
- net GND: now also C11.2, C13.-, J3.GND, U5.AGND, U5.GND, U5.TEST
- net RXD: now also U5.TXD
- net TXD: now also U5.RXD

Commit message: Add files via upload
Parts:
- added B2: (no value), ME507:BEAD0805
- added C14, C15: 22pF, rcl:C-USC0805
- added C16: 4.7uF, rcl:CPOL-USA/3216-18W
- added C17: 100nF, rcl:C-USC0805
- added R10, R11: 270, rcl:R-US_R0805
- added R2: 4.7k, rcl:R-US_R0805
- added R3: 330, rcl:R-US_R0805
- added R4, R5: (no value), rcl:R-US_R0805
- added R6: 100m, rcl:R-US_R0805
- added R7, R8, R9: 500, rcl:R-US_R0805
- added SW1: SW, ME507:SW
- added U$1, U$10, U$11, U$12, U$13, U$2, U$3, U$4, U$5, U$6, U$7, U$8, U$9: NC, ME507:NC
- added Y2: 30MHz, Downloads:ECS-160-20-3X-TR
- C6, C7: value 22pF -> 20pF
- R1: value 200m -> 400m
Connections:
- net N$4 renamed DP
- net N$5 renamed DM
- removed net !SLEEP!: U2.!SLEEP!
- removed net 3V3: C11.1, U5.3V3OUT
- removed net N$2: B1.1, U5.VCC, U5.VCCIO
- removed net N$3: R1.1, U2.AISEN, U2.BISEN
- new net +3V3: C11.1, JP4.4, R4.1, R5.1, U5.3V3OUT
- new net AISEN: R6.1, U2.AISEN
- new net AVCC: B2.1, C10.1, U1.AVCC
- new net BISEN: R1.1, U2.BISEN
- new net BUS0: R11.2, U5.CBUS0
- new net BUS1: R10.2, U5.CBUS1
- new net FCKI: C14.1, U3.FCKI, Y2.1
- new net FCKO: C15.1, U3.FCKO, Y2.2
- new net MI: R9.2, U3.MISO
- new net MO: R8.2, U3.MOSI
- new net N$12: J3.ID, U$1.D
- new net N$16: U$2.D, U5.OSCI
- new net N$17: U$3.D, U5.OSCO
- new net N$18: U$4.D, U5.!RESET
- new net N$20: U$5.D, U5.!DSR
- new net N$21: U$6.D, U5.!RI
- new net N$22: U$7.D, U5.!DCD
- new net N$23: U$8.D, U5.!DTR
- new net N$24: U$9.D, U5.CBUS2
- new net N$25: U$10.D, U5.CBUS3
- new net N$26: U$11.D, U5.CBUS4
- new net N$27: U$12.D, U3.INDEX/
- new net N$28: U$13.D, U3.DFLAG/
- new net SCK: JP1.3, R7.1, U1.PB5
- new net SW: R3.1, SW1.S
- new net VCCIO: B1.1, C16.+, R10.1, R11.1, U5.VCC, U5.VCCIO
- net !RESET!: now also C17.1, R2.1, R3.2
- net !SS!: now also U1.PD2; no longer U1.PB5
- net +5V: now also B2.2, R2.2, U2.!SLEEP!; no longer C10.1, U1.AVCC
- net AIN1: now also U1.PD5; no longer U1.PD3
- net AIN2: now also U1.PD6; no longer U1.PD5
- net BIN1: now also U1.PB1; no longer U1.PD6
- net BIN2: now also U1.PB2; no longer U1.PB1
- net ENCA: now also JP4.3, R4.2; no longer JP4.4
- net ENCB: now also JP4.2, R5.2; no longer JP4.3
- net GND: now also C14.2, C15.2, C16.-, C17.2, JP4.1, R6.2, SW1.P, U3.VSS
- net MISO: now also R9.1, U1.PB4; no longer U1.PB3, U3.MISO
- net MOSI: now also R8.1, U1.PB3; no longer U1.PB4, U3.MOSI
- net SCLK: now also R7.2; no longer JP1.3, U1.PB2
Other:
- note added: "LEDs here"
- moved on the sheet: B1, C10, C11, C3, C4, C5, C6, C7, J3, JP3, JP4, Y1

Commit message: Add files via upload
Parts:
- added D1: HSMC-C190, HSMC-C190:HSMC-C190
- added S1: 5-1437565-0, 5-1437565-0:5-1437565-0
- C1, C10, C11, C12, C17, C2, C4, C5, C8, C9: device rcl:C-USC0805 -> C2012X7R1V225K125AE:C2012X7R1V225K125AE
- C14, C15, C6, C7: device rcl:C-USC0805 -> 101X15N220MV4E:101X15N220MV4E
- R1: device rcl:R-US_R0805 -> RL1206FR-070R4L:RL1206FR-070R4L
Other:
- note added: "LED"
- note added: "STILL NEEDED"
- moved on the sheet: C1, C10, C11, C12, C14, C15, C17, C2, C4, C5, C6, C7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

Commit message: Add files via upload
Parts:
- removed D1: HSMC-C190, HSMC-C190:HSMC-C190
- removed SW1: SW, ME507:SW
- added U$14, U$15, U$16: NC, ME507:NC
- C1, C10, C11, C12, C17, C2, C4, C5, C8, C9: device C2012X7R1V225K125AE:C2012X7R1V225K125AE -> rcl:C-USC0805
- C14, C15: value 22pF -> 20pF; device 101X15N220MV4E:101X15N220MV4E -> rcl:C-USC0805
- C6, C7: device 101X15N220MV4E:101X15N220MV4E -> rcl:C-USC0805
- R1: device RL1206FR-070R4L:RL1206FR-070R4L -> rcl:R-US_R0805
- S1: device 5-1437565-0:5-1437565-0 -> Downloads:5-1437565-0
Connections:
- new net LFLAG: U1.PD4, U3.LFLAG/
- new net N$2: U$14.D, U5.!RTS
- new net N$3: U$15.D, U5.!CTS
- new net N$4: U$16.D, U3.CNT_EN
- net !FAULT!: now also U1.PD3
- net GND: now also S1.1; no longer SW1.P
- net SW: now also S1.2; no longer SW1.S
Other:
- note added: "RXLED"
- note added: "Reset Switch"
- note added: "Sensor Header"
- note added: "TXLED"
- note added: "UART Bridge"
- note removed: "LED"
- note removed: "LEDs here"
- note removed: "STILL NEEDED"
- moved on the sheet: B1, B2, C1, C10, C11, C12, C13, C14, C15, C16, C17, C2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
