File: main.sch (EAGLE design)
At the start: 60 parts, among them J1 PJ-015AH-SMT-TR, J3 1734510-1, U1 ATMEGA328P-AU, U2 DRV8833PWPR, U3 LS7366R-TS, U4 LP38691DTX-5.0/NOPB, U5 FT232RL-REEL, Y1 16MHz, Y2 30MHz

Commit message: Add files via upload
Parts:
- added D1: RED LED, HSMC-C190:HSMC-C190
- added D2, D3: GREEN LED, HSMC-C190:HSMC-C190
- added R14: 270, rcl:R-US_R0805
Connections:
- new net N$5: R14.2, U1.ADC6
- new net N$6: D1.A, R14.1
- new net N$7: D3.A, R11.1
- net GND: now also D1.C, D2.C, D3.C
- net VCCIO: now also D2.A; no longer R11.1
Other:
- note removed: "RXLED"
- note removed: "TXLED"
Changed lines of the file:
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@@
 <drawing>
 <settings>
-<setting alwaysvectorfont="no"/>
+<setting alwaysvectorfont="yes"/>
 <setting verticaltext="up"/>
 </settings>
@@
 <part name="U$15" library="ME507" deviceset="NC" device=""/>
 <part name="U$16" library="ME507" deviceset="NC" device=""/>
+<part name="R14" library="rcl" library_urn="urn:adsk.eagle:library:334" deviceset="R-US_" device="R0805" package3d_urn="urn:adsk.eagle:package:23553/2" value="270"/>
+<part name="D1" library="HSMC-C190" deviceset="HSMC-C190" device="" value="RED LED"/>
+<part name="GND27" library="supply1" library_urn="urn:adsk.eagle:library:371" deviceset="GND" device=""/>
+<part name="D2" library="HSMC-C190" deviceset="HSMC-C190" device="" value="GREEN LED"/>
+<part name="D3" library="HSMC-C190" deviceset="HSMC-C190" device="" value="GREEN LED"/>
+<part name="GND28" library="supply1" library_urn="urn:adsk.eagle:library:371" deviceset="GND" device=""/>
+<part name="GND29" library="supply1" library_urn="urn:adsk.eagle:library:371" deviceset="GND" device=""/>
 </parts>
 <sheets>
@@
 <attribute name="VALUE" x="27.938459375" y="68.83253125" size="1.778540625" layer="96"/>
 </instance>
+<instance part="R14" gate="G$1" x="167.64" y="121.92" smashed="yes" rot="R180">
+<attribute name="NAME" x="171.45" y="120.4214" size="1.778" layer="95" rot="R180"/>
+<attribute name="VALUE" x="171.45" y="125.222" size="1.778" layer="96" rot="R180"/>
+</instance>
+<instance part="D1" gate="G$1" x="190.5" y="121.92" smashed="yes" rot="R180">
+<attribute name="NAME" x="192.53513125" y="117.84973125" size="1.780740625" layer="95" rot="R180"/>
+<attribute name="VALUE" x="192.53368125" y="125.73315" size="1.77946875" layer="96" rot="R180"/>
+</instance>
+<instance part="GND27" gate="1" x="203.2" y="114.3" smashed="yes">
+<attribute name="VALUE" x="200.66" y="111.76" size="1.778" layer="96"/>
+</instance>
 </instances>
 <busses>
@@
 <pinref part="GND26" gate="1" pin="GND"/>
 <wire x1="55.88" y1="63.5" x2="55.88" y2="60.96" width="0.1524" layer="91"/>
+</segment>
+<segment>
+<pinref part="D1" gate="G$1" pin="C"/>
+<wire x1="198.12" y1="121.92" x2="203.2" y2="121.92" width="0.1524" layer="91"/>
+<pinref part="GND27" gate="1" pin="GND"/>
+<wire x1="203.2" y1="121.92" x2="203.2" y2="116.84" width="0.1524" layer="91"/>
 </segment>
 </net>
@@
 <wire x1="167.64" y1="139.7" x2="170.18" y2="139.7" width="0.1524" layer="91"/>
 <label x="170.18" y="139.7" size="1.778" layer="95" xref="yes"/>
+</segment>
+</net>
+<net name="N$5" class="0">
+<segment>
+<pinref part="U1" gate="G$1" pin="ADC6"/>
+<wire x1="144.78" y1="129.54" x2="157.48" y2="129.54" width="0.1524" layer="91"/>
+<wire x1="157.48" y1="129.54" x2="157.48" y2="121.92" width="0.1524" layer="91"/>
+<pinref part="R14" gate="G$1" pin="2"/>
+<wire x1="157.48" y1="121.92" x2="162.56" y2="121.92" width="0.1524" layer="91"/>
+</segment>
+</net>
+<net name="N$6" class="0">
+<segment>
+<pinref part="R14" gate="G$1" pin="1"/>
+<pinref part="D1" gate="G$1" pin="A"/>
+<wire x1="172.72" y1="121.92" x2="180.34" y2="121.92" width="0.1524" layer="91"/>
 </segment>
 </net>
@@
 <description>USB to UART</description>
 <plain>
-<text x="40.64" y="76.2" size="1.778" layer="150">TXLED</text>
-<text x="40.64" y="68.58" size="1.778" layer="150">RXLED</text>
 <text x="175.26" y="114.3" size="1.778" layer="95">Voltage Regulator</text>
 <text x="86.36" y="162.56" size="1.778" layer="150">UART Bridge</text>
@@
 <attribute name="VALUE" x="213.36" y="109.22" size="1.778" layer="96" rot="R180"/>
 </instance>
+<instance part="D2" gate="G$1" x="50.8" y="55.88" smashed="yes" rot="R90">
+<attribute name="NAME" x="46.72973125" y="53.84486875" size="1.780740625" layer="95" rot="R90"/>
+<attribute name="VALUE" x="54.61315" y="53.84631875" size="1.77946875" layer="96" rot="R90"/>
+</instance>
+<instance part="D3" gate="G$1" x="40.64" y="55.88" smashed="yes" rot="R90">
+<attribute name="NAME" x="36.56973125" y="53.84486875" size="1.780740625" layer="95" rot="R90"/>
+<attribute name="VALUE" x="44.45315" y="53.84631875" size="1.77946875" layer="96" rot="R90"/>
+</instance>
+<instance part="GND28" gate="1" x="40.64" y="40.64" smashed="yes">
+<attribute name="VALUE" x="38.1" y="38.1" size="1.778" layer="96"/>
+</instance>
+<instance part="GND29" gate="1" x="50.8" y="40.64" smashed="yes">
+<attribute name="VALUE" x="48.26" y="38.1" size="1.778" layer="96"/>
+</instance>
 </instances>
 <busses>
@@
 <wire x1="210.82" y1="104.14" x2="210.82" y2="101.6" width="0.1524" layer="91"/>
 <junction x="210.82" y="101.6"/>
+</segment>
+<segment>
+<pinref part="D3" gate="G$1" pin="C"/>
+<pinref part="GND28" gate="1" pin="GND"/>
+<wire x1="40.64" y1="48.26" x2="40.64" y2="43.18" width="0.1524" layer="91"/>
+</segment>
+<segment>
+<pinref part="D2" gate="G$1" pin="C"/>
+<pinref part="GND29" gate="1" pin="GND"/>
+<wire x1="50.8" y1="48.26" x2="50.8" y2="43.18" width="0.1524" layer="91"/>
 </segment>
 </net>
@@
 </segment>
 <segment>
-<label x="40.64" y="71.12" size="1.778" layer="95"/>
 <pinref part="R10" gate="G$1" pin="1"/>
-<wire x1="50.8" y1="71.12" x2="40.64" y2="71.12" width="0.1524" layer="91"/>
-<wire x1="50.8" y1="83.82" x2="50.8" y2="71.12" width="0.1524" layer="91"/>
 <wire x1="50.8" y1="83.82" x2="53.34" y2="83.82" width="0.1524" layer="91"/>
-</segment>
-<segment>
-<pinref part="R11" gate="G$1" pin="1"/>
-<wire x1="53.34" y1="93.98" x2="48.26" y2="93.98" width="0.1524" layer="91"/>
-<wire x1="48.26" y1="93.98" x2="48.26" y2="78.74" width="0.1524" layer="91"/>
-<wire x1="48.26" y1="78.74" x2="40.64" y2="78.74" width="0.1524" layer="91"/>
-<label x="40.64" y="78.74" size="1.778" layer="95"/>
+<pinref part="D2" gate="G$1" pin="A"/>
+<wire x1="50.8" y1="83.82" x2="50.8" y2="66.04" width="0.1524" layer="91"/>
 </segment>
 </net>
@@
 </segment>
 </net>
+<net name="N$7" class="0">
+<segment>
+<pinref part="R11" gate="G$1" pin="1"/>
+<wire x1="53.34" y1="93.98" x2="40.64" y2="93.98" width="0.1524" layer="91"/>
+<pinref part="D3" gate="G$1" pin="A"/>
+<wire x1="40.64" y1="93.98" x2="40.64" y2="66.04" width="0.1524" layer="91"/>
+</segment>
+</net>

Commit message: Add files via upload
Parts:
- C16: device rcl:CPOL-USA/3216-18W -> rcl:CPOL-USE5-5
- C3: device rcl:CPOL-US153CLV-0605 -> rcl:CPOL-USE5-4
Changed lines of the file:
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@@
 <part name="C2" library="rcl" library_urn="urn:adsk.eagle:library:334" deviceset="C-US" device="C0805" package3d_urn="urn:adsk.eagle:package:23617/2" value="10nF"/>
 <part name="R1" library="rcl" library_urn="urn:adsk.eagle:library:334" deviceset="R-US_" device="R0805" package3d_urn="urn:adsk.eagle:package:23553/2" value="400m"/>
-<part name="C3" library="rcl" library_urn="urn:adsk.eagle:library:334" deviceset="CPOL-US" device="153CLV-0605" package3d_urn="urn:adsk.eagle:package:23398/2" value="10uF"/>
+<part name="C3" library="rcl" library_urn="urn:adsk.eagle:library:334" deviceset="CPOL-US" device="E5-4" package3d_urn="urn:adsk.eagle:package:23370/1" value="10uF"/>
 <part name="GND4" library="supply1" library_urn="urn:adsk.eagle:library:371" deviceset="GND" device=""/>
 <part name="U2" library="Downloads" deviceset="DRV8833PWPR" device=""/>
@@
 <part name="C15" library="rcl" library_urn="urn:adsk.eagle:library:334" deviceset="C-US" device="C0805" package3d_urn="urn:adsk.eagle:package:23617/2" value="20pF"/>
 <part name="GND23" library="supply1" library_urn="urn:adsk.eagle:library:371" deviceset="GND" device=""/>
-<part name="C16" library="rcl" library_urn="urn:adsk.eagle:library:334" deviceset="CPOL-US" device="A/3216-18W" package3d_urn="urn:adsk.eagle:package:23408/2" value="4.7uF"/>
+<part name="C16" library="rcl" library_urn="urn:adsk.eagle:library:334" deviceset="CPOL-US" device="E5-5" package3d_urn="urn:adsk.eagle:package:23367/2" value="4.7uF"/>
 <part name="GND24" library="supply1" library_urn="urn:adsk.eagle:library:371" deviceset="GND" device=""/>
 <part name="R6" library="rcl" library_urn="urn:adsk.eagle:library:334" deviceset="R-US_" device="R0805" package3d_urn="urn:adsk.eagle:package:23553/2" value="100m"/>

Commit message: Add files via upload
Connections:
- net DM renamed N$9
- net DP renamed N$10
- removed net N$7: D3.A, R11.1
- new net RXLED: D2.C, R10.1
- new net TXLED: D3.C, R11.1
- net FLOW: now also U1.PB0
- net GND: now also R14.1; no longer D1.C, D2.C, D3.C
- net N$5: now also D1.A, U1.PD7; no longer R14.2, U1.ADC6
- net N$6: now also D1.C, R14.2; no longer D1.A, R14.1
- net VCCIO: now also D3.A; no longer R10.1
Other:
- note added: "Decoupling Capacitors"
- note added: "Motor driver input 2.7 - 10.8V"
- note added: "Unsure about the value of the ferrite bead [B1]"
- note added: "Unsure about the value of the ferrite bead [B2]"
- note added: "Voltage regulator input 2.7 - 10V"
- note removed: "VCC Decoupling Capacitors"
- moved on the sheet: C12, C13, C6, C7, D1, D2, D3, J3, R14, Y1

Commit message: Add files via upload
Parts:
- added R12: 1M, rcl:R-US_R0805
- C13: device rcl:CPOL-USA/3216-18W -> rcl:C-USC0805
- JP2: device pinhead:PINHD-2X4 -> Downloads:PINHD-2X4
- JP3, JP4: device pinhead:PINHD-1X4 -> Downloads:PINHD-1X4
Connections:
- removed net ENCA: JP4.3, R4.2, U3.A
- removed net ENCB: JP4.2, R5.2, U3.B
- new net N$7: JP4.3, R5.2, U3.B
- new net N$8: JP4.2, R4.2, U3.A
- net FCKI: now also R12.2
- net FCKO: now also R12.1
- net GND: now also C13.2; no longer C13.-
- net VCC: now also C13.1; no longer C13.+
Other:
- moved on the sheet: C14, C15, JP4, Y2

Commit message: Add files via upload
Parts:
- B1, B2: value (none) -> 100
- J1: value PJ-015AH-SMT-TR -> PJ-036AH-SMT-TR; device Downloads:PJ-015AH-SMT-TR -> Downloads:PJ-036AH-SMT-TR
- R4, R5: value (none) -> 4.7
- U3: value LS7366R-TS -> LS7366R-S; device Downloads:LS7366R-TS -> Downloads:LS7366R-TSLS7366R-S
Connections:
- net N$10 renamed DP
- net N$5 renamed PD7
- net N$6 renamed LED
- net N$7 renamed ENCB
- net N$8 renamed ENCA
- net N$9 renamed DM
Changed lines of the file:
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@@
 <part name="GND9" library="supply1" library_urn="urn:adsk.eagle:library:371" deviceset="GND" device=""/>
 <part name="P+4" library="supply1" library_urn="urn:adsk.eagle:library:371" deviceset="+5V" device=""/>
-<part name="U3" library="Downloads" deviceset="LS7366R-TS" device=""/>
+<part name="U3" library="Downloads" deviceset="LS7366R-TS" device="LS7366R-S" package3d_urn="urn:adsk.eagle:package:14910052/1" value="LS7366R-S"/>
 <part name="P+5" library="supply1" library_urn="urn:adsk.eagle:library:371" deviceset="+5V" device=""/>
 <part name="Y1" library="Downloads" deviceset="ECS-160-20-3X-TR" device="" value="16MHz"/>
-<part name="J1" library="Downloads" deviceset="PJ-015AH-SMT-TR" device=""/>
+<part name="J1" library="Downloads" deviceset="PJ-036AH-SMT-TR" device=""/>
 <part name="JP1" library="pinhead" library_urn="urn:adsk.eagle:library:325" deviceset="PINHD-2X3" device="" package3d_urn="urn:adsk.eagle:package:22462/2"/>
 <part name="P+6" library="supply1" library_urn="urn:adsk.eagle:library:371" deviceset="+5V" device=""/>
@@
 <part name="GND15" library="supply1" library_urn="urn:adsk.eagle:library:371" deviceset="GND" device=""/>
 <part name="GND16" library="supply1" library_urn="urn:adsk.eagle:library:371" deviceset="GND" device=""/>
-<part name="B1" library="ME507" deviceset="BEAD" device="0805"/>
+<part name="B1" library="ME507" deviceset="BEAD" device="0805" value="100"/>
 <part name="GND17" library="supply1" library_urn="urn:adsk.eagle:library:371" deviceset="GND" device=""/>
 <part name="GND18" library="supply1" library_urn="urn:adsk.eagle:library:371" deviceset="GND" device=""/>
 <part name="C13" library="rcl" library_urn="urn:adsk.eagle:library:334" deviceset="C-US" device="C0805" package3d_urn="urn:adsk.eagle:package:23617/2" value="10nF"/>
-<part name="B2" library="ME507" deviceset="BEAD" device="0805"/>
+<part name="B2" library="ME507" deviceset="BEAD" device="0805" value="100"/>
 <part name="P+7" library="supply1" library_urn="urn:adsk.eagle:library:371" deviceset="+5V" device=""/>
 <part name="P+8" library="ME507" deviceset="AVCC" device=""/>
@@
 <part name="+3V1" library="supply1" library_urn="urn:adsk.eagle:library:371" deviceset="+3V3" device=""/>
 <part name="+3V2" library="supply1" library_urn="urn:adsk.eagle:library:371" deviceset="+3V3" device=""/>
-<part name="R4" library="rcl" library_urn="urn:adsk.eagle:library:334" deviceset="R-US_" device="R0805" package3d_urn="urn:adsk.eagle:package:23553/2"/>
-<part name="R5" library="rcl" library_urn="urn:adsk.eagle:library:334" deviceset="R-US_" device="R0805" package3d_urn="urn:adsk.eagle:package:23553/2"/>
+<part name="R4" library="rcl" library_urn="urn:adsk.eagle:library:334" deviceset="R-US_" device="R0805" package3d_urn="urn:adsk.eagle:package:23553/2" value="4.7"/>
+<part name="R5" library="rcl" library_urn="urn:adsk.eagle:library:334" deviceset="R-US_" device="R0805" package3d_urn="urn:adsk.eagle:package:23553/2" value="4.7"/>
 <part name="+3V3" library="supply1" library_urn="urn:adsk.eagle:library:371" deviceset="+3V3" device=""/>
 <part name="+3V4" library="supply1" library_urn="urn:adsk.eagle:library:371" deviceset="+3V3" device=""/>
@@
 </instance>
 <instance part="B2" gate="G$1" x="210.82" y="78.74" smashed="yes" rot="R90">
-<attribute name="NAME" x="207.01" y="74.93" size="1.778" layer="95"/>
-<attribute name="VALUE" x="217.17" y="74.93" size="1.778" layer="96" rot="R90"/>
+<attribute name="NAME" x="212.09" y="80.01" size="1.778" layer="95"/>
+<attribute name="VALUE" x="214.63" y="77.47" size="1.778" layer="96"/>
 </instance>
 <instance part="P+7" gate="1" x="210.82" y="88.9" smashed="yes">
@@
 <attribute name="VALUE" x="144.78" y="167.64" size="1.778" layer="96"/>
 </instance>
-<instance part="P+9" gate="AVCC" x="220.98" y="78.74" smashed="yes">
-<attribute name="VALUE" x="218.44" y="78.74" size="1.778" layer="96"/>
+<instance part="P+9" gate="AVCC" x="220.98" y="88.9" smashed="yes">
+<attribute name="VALUE" x="218.44" y="88.9" size="1.778" layer="96"/>
 </instance>
 <instance part="GND19" gate="1" x="210.82" y="55.88" smashed="yes" rot="MR0">
@@
 <junction x="210.82" y="71.12"/>
 <pinref part="P+9" gate="AVCC" pin="AVCC"/>
-<wire x1="220.98" y1="71.12" x2="220.98" y2="76.2" width="0.1524" layer="91"/>
+<wire x1="220.98" y1="71.12" x2="220.98" y2="86.36" width="0.1524" layer="91"/>
 </segment>
 </net>
@@
 </segment>
 </net>
-<net name="N$5" class="0">
+<net name="PD7" class="0">
 <segment>
 <pinref part="U1" gate="G$1" pin="PD7"/>
@@
 </segment>
 </net>
-<net name="N$6" class="0">
+<net name="LED" class="0">
 <segment>
 <pinref part="D1" gate="G$1" pin="C"/>
@@
 </instance>
 <instance part="R5" gate="G$1" x="177.8" y="104.14" smashed="yes" rot="MR270">
-<attribute name="NAME" x="178.8414" y="107.95" size="1.778" layer="95" rot="MR180"/>
-<attribute name="VALUE" x="176.022" y="102.87" size="1.778" layer="96" rot="MR0"/>
+<attribute name="NAME" x="179.2986" y="107.95" size="1.778" layer="95" rot="MR180"/>
+<attribute name="VALUE" x="179.578" y="102.87" size="1.778" layer="96" rot="MR180"/>
 </instance>
 <instance part="+3V3" gate="G$1" x="170.18" y="114.3" smashed="yes">
@@
 </segment>
 </net>
-<net name="N$7" class="0">
+<net name="ENCB" class="0">
 <segment>
 <pinref part="JP4" gate="A" pin="3"/>
@@
 </segment>
 </net>
-<net name="N$8" class="0">
+<net name="ENCA" class="0">
 <segment>
 <pinref part="U3" gate="G$1" pin="A"/>
@@
 <instance part="B1" gate="G$1" x="121.92" y="157.48" smashed="yes" rot="R90">
 <attribute name="NAME" x="123.19" y="158.75" size="1.778" layer="95"/>
-<attribute name="VALUE" x="128.27" y="153.67" size="1.778" layer="96" rot="R90"/>
+<attribute name="VALUE" x="125.73" y="156.21" size="1.778" layer="96"/>
 </instance>
 <instance part="GND17" gate="1" x="40.64" y="134.62" smashed="yes" rot="R180">
@@
 </segment>
 </net>
-<net name="N$9" class="0">
+<net name="DM" class="0">
 <segment>
 <pinref part="J3" gate="G$1" pin="D-"/>
@@
 </segment>
 </net>
-<net name="N$10" class="0">
+<net name="DP" class="0">
 <segment>
 <pinref part="U5" gate="G$1" pin="USBDP"/>

Commit message: Add files via upload
Parts:
- B1, B2: DIGIKEYPART# (none) -> ‎240-2395-1-ND‎
- C1: DIGIKEYPART# (none) -> ‎311-3507-1-ND‎
- C10, C11, C12, C17, C8, C9: DIGIKEYPART# (none) -> ‎311-1361-1-ND‎
- C13, C2: DIGIKEYPART# (none) -> ‎311-1136-1-ND‎
- C14, C15, C6, C7: DIGIKEYPART# (none) -> ‎311-4221-1-ND‎
- C16: DIGIKEYPART# (none) -> ‎493-6100-1-ND‎
- C3: DIGIKEYPART# (none) -> ‎493-13387-ND‎
- C4, C5: DIGIKEYPART# (none) -> ‎311-1358-1-ND‎
- R1: DIGIKEYPART# (none) -> P390ADCT-ND‎
- R10, R11, R14: DIGIKEYPART# (none) -> RHM270KCT-ND‎
- R12: DIGIKEYPART# (none) -> A102079CT-ND‎
- R2, R4, R5, R7, R8, R9: DIGIKEYPART# (none) -> ‎A129546CT-ND‎
- R3: DIGIKEYPART# (none) -> ‎P330ADCT-ND‎
- R6: DIGIKEYPART# (none) -> ‎RNCP0805FTD100RCT-ND‎

Commit message: Add files via upload
Parts:
- B1: DIGIKEYPART# ‎240-2395-1-ND‎ -> (none)
- B2: value 100 -> 120; DIGIKEYPART# ‎240-2395-1-ND‎ -> (none)
- C1: DIGIKEYPART# ‎311-3507-1-ND‎ -> (none)
- C10, C11, C12, C17, C8, C9: DIGIKEYPART# ‎311-1361-1-ND‎ -> (none)
- C13, C2: DIGIKEYPART# ‎311-1136-1-ND‎ -> (none)
- C14, C15, C6, C7: DIGIKEYPART# ‎311-4221-1-ND‎ -> (none)
- C16: DIGIKEYPART# ‎493-6100-1-ND‎ -> (none)
- C3: DIGIKEYPART# ‎493-13387-ND‎ -> (none)
- C4, C5: DIGIKEYPART# ‎311-1358-1-ND‎ -> (none)
- R1: DIGIKEYPART# P390ADCT-ND‎ -> (none)
- R10, R11, R14: DIGIKEYPART# RHM270KCT-ND‎ -> (none)
- R12: DIGIKEYPART# A102079CT-ND‎ -> (none)
- R2, R7, R8, R9: DIGIKEYPART# ‎A129546CT-ND‎ -> (none)
- R3: DIGIKEYPART# ‎P330ADCT-ND‎ -> (none)
- R4, R5: value 4.7 -> 4.7k; DIGIKEYPART# ‎A129546CT-ND‎ -> (none)
- R6: DIGIKEYPART# ‎RNCP0805FTD100RCT-ND‎ -> (none)
Other:
- note removed: "Unsure about the value of the ferrite bead [B1]"
- note removed: "Unsure about the value of the ferrite bead [B2]"
